Commit message: refactor

File: urdf/two_wheels.urdf.xacro (robot description, xacro)
@@ -2,5 +2,4 @@
 <robot xmlns:xacro="http://wiki.ros.org/xacro" name="two_wheels">
   <!-- Use this if parameters are set from the launch file, otherwise delete -->
-  <xacro:arg name="prefix" default="" />
   <xacro:arg name="use_mock_hardware" default="false" />
   <xacro:arg name="mock_sensor_commands" default="false" />
@@ -10,14 +9,9 @@
   <xacro:include filename="$(find two_wheels)/urdf/two_wheels/two_wheels_macro.xacro"/>
   <xacro:include filename="$(find two_wheels)/urdf/two_wheels/two_wheels_macro.ros2_control.xacro"/>
-  <!-- create link fixed to the "world" -->
-  <link name="world" />
   <!-- Load robot's macro with parameters -->
-  <!-- set prefix if multiple robots are used -->
-  <xacro:two_wheels prefix="$(arg prefix)" parent="world" >
-    <origin xyz="0 0 0" rpy="0 0 0" />          <!-- position robot in the world -->
+  <xacro:two_wheels>
   </xacro:two_wheels>
   <xacro:two_wheels_ros2_control
     name="two_wheels"
-    prefix="$(arg prefix)"
     use_mock_hardware="$(arg use_mock_hardware)"
     mock_sensor_commands="$(arg mock_sensor_commands)"

File: urdf/two_wheels/two_wheels_macro.ros2_control.xacro (robot description, xacro)
@@ -3,5 +3,4 @@
   <xacro:macro name="two_wheels_ros2_control" params="
                name
-               prefix
                use_mock_hardware:=^|false
                mock_sensor_commands:=^|false
@@ -53,15 +52,4 @@
       </gazebo>
     </xacro:if>
-    <xacro:if value="$(arg sim_gazebo)">
-      <!-- Gazebo plugins -->
-      <gazebo reference="world">
-      </gazebo>
-      <gazebo>
-        <plugin filename="libign_ros2_control-system.so" name="ign_ros2_control::IgnitionROS2ControlPlugin">
-          <parameters>${simulation_controllers}</parameters>
-          <controller_manager_node_name>${prefix}controller_manager</controller_manager_node_name>
-        </plugin>
-      </gazebo>
-    </xacro:if>
   </xacro:macro>
 </robot>

File: urdf/two_wheels/two_wheels_macro.xacro (robot description, xacro)
@@ -38,13 +38,13 @@
             <parent link="base_link"/>
             <child link="${prefix}_wheel"/>
-            <origin xyz="0 ${y_reflect*(disc_radius+(wheel_width/2))} 0" rpy="0 0 0"/>
+            <origin xyz="0 ${y_reflect*(disc_radius+(wheel_width/2))} ${wheel_radius}" rpy="0 0 0"/>
             <axis xyz="0 1 0"/>
         </joint>
     </xacro:macro>
-    <xacro:macro name="two_wheels" params="prefix parent *origin">
+    <xacro:macro name="two_wheels" >
         <link name="base_link">
             <xacro:cylinder_inertial mass="${disc_mass}" radius="${disc_radius}" length="${disc_height}" rotation="0"/>
             <visual>
-                <origin xyz="0 0 0" rpy="0 0 0"/>
+                <origin xyz="0 0 ${wheel_radius}" rpy="0 0 0"/>
                 <geometry>
                     <cylinder radius="${disc_radius}" length="${disc_height}"/>
@@ -59,9 +59,9 @@
             </collision>
         </link>
-        <joint name="base_joint" type="fixed">
-            <parent link="world"/>
-            <child link="base_link"/>
-            <origin xyz="0.0 0.0 ${-wheel_radius}" rpy="0 0 0"/>
-        </joint>
+<!--        <joint name="base_joint" type="fixed">-->
+<!--            <parent link="base_footprint"/>-->
+<!--            <child link="base_link"/>-->
+<!--            <origin xyz="0.0 0.0 ${-wheel_radius}" rpy="0 0 0"/>-->
+<!--        </joint>-->
         <xacro:wheel prefix="left" y_reflect="1"/>
         <xacro:wheel prefix="right" y_reflect="-1"/>

Commit message: gazebo

File: urdf/two_wheels.urdf.xacro (robot description, xacro)
@@ -1,5 +1,4 @@
 <?xml version="1.0" encoding="UTF-8"?>
 <robot xmlns:xacro="http://wiki.ros.org/xacro" name="two_wheels">
-  <!-- Use this if parameters are set from the launch file, otherwise delete -->
   <xacro:arg name="use_mock_hardware" default="false" />
   <xacro:arg name="mock_sensor_commands" default="false" />

File: urdf/two_wheels/two_wheels_macro.xacro (robot description, xacro)
@@ -66,4 +66,13 @@
         <xacro:wheel prefix="left" y_reflect="1"/>
         <xacro:wheel prefix="right" y_reflect="-1"/>
+        <gazebo reference="base_link">
+            <material>Gazebo/White</material>
+        </gazebo>
+        <gazebo reference="left_wheel">
+            <material>Gazebo/Black</material>
+        </gazebo>
+        <gazebo reference="right_wheel">
+            <material>Gazebo/Black</material>
+        </gazebo>
     </xacro:macro>
 </robot>
