Commit message: added sonar

File: urdf/robot.urdf.xacro (robot description, xacro)
@@ -2,4 +2,5 @@
 <robot xmlns:xacro="http://www.ros.org/wiki/xacro" name="robot">
     <xacro:include filename="robot_core.xacro"/>
+    <xacro:include filename="sonar.xacro"/>
     <xacro:if value="$(arg is_sim)">
         <xacro:include filename="gazebo_control.xacro"/>

File: urdf/robot_core.xacro (robot description, xacro)
@@ -14,4 +14,5 @@
     <xacro:property name="caster_wheel_offset_x" value="0.06"/>
     <xacro:property name="caster_wheel_offset_z" value="${caster_wheel_radius}"/>
+    <xacro:property name="sonar_size" value="0.01"/>
     <material name="white">
         <color rgba="1.0 1.0 1.0 1.0"/>
@@ -23,4 +24,7 @@
         <color rgba="0 0 0 1"/>
     </material>
+    <material name="cyan">
+        <color rgba="0 1 1 1"/>
+    </material>
     <xacro:macro name="wheel" params="prefix y_reflect">
         <link name="${prefix}_wheel">
@@ -30,6 +34,5 @@
                     <cylinder radius="${wheel_radius}" length="${wheel_width}"/>
                 </geometry>
-                <material name="black">
-                </material>
+                <material name="black"/>
             </visual>
             <collision>
@@ -94,3 +97,16 @@
         <origin xyz="${caster_wheel_offset_x} 0 -${caster_wheel_offset_z}"/>
     </joint>
+    <link name="sonar_link">
+        <visual>
+            <geometry>
+                <box size="${sonar_size} ${sonar_size} ${sonar_size}"/>
+            </geometry>
+            <material name="cyan"/>
+        </visual>
+    </link>
+    <joint name="sonar_link_joint" type="fixed">
+        <parent link="base_link"/>
+        <child link="sonar_link"/>
+        <origin xyz="${caster_wheel_offset_x}  0 0"/>
+    </joint>
 </robot>

Commit message: added lidar link

File: urdf/robot.urdf.xacro (robot description, xacro)
@@ -7,4 +7,5 @@
         <xacro:include filename="gazebo/sonar.xacro"/>
         <xacro:include filename="gazebo/imu.xacro"/>
+        <xacro:include filename="gazebo/lidar.xacro"/>
     </xacro:if>
     <xacro:unless value="$(arg is_sim)">

File: urdf/robot_core.xacro (robot description, xacro)
@@ -145,3 +145,30 @@
         <axis xyz="0 0 0"/>
     </joint>
+    <link name="lidar_link">
+        <visual>
+            <geometry>
+                <cylinder radius="0.05" length="0.04"/>
+            </geometry>
+            <material name="black"/>
+        </visual>
+        <visual>
+            <origin xyz="0 0 -0.05"/>
+            <geometry>
+                <cylinder radius="0.01" length="0.1"/>
+            </geometry>
+            <material name="black"/>
+        </visual>
+        <collision>
+            <geometry>
+                <cylinder radius="0.05" length="0.04"/>
+            </geometry>
+        </collision>
+        <xacro:cylinder_inertial mass="0.1" radius="0.04" length="0.05" rotation="0"/>
+    </link>
+    <joint name="lidar_joint" type="fixed">
+        <origin xyz="0 0 0" rpy="0 0 0"/>
+        <parent link="base_link"/>
+        <child link="lidar_link"/>
+        <axis xyz="0 0 0"/>
+    </joint>
 </robot>
