Commit message: sonar_link_joint z position to 0

File: urdf/robot_core.xacro (robot description, xacro)
@@ -116,5 +116,5 @@
         <parent link="base_link"/>
         <child link="sonar_link"/>
-        <origin xyz="${disc_radius} 0 0.01"/>
+        <origin xyz="${disc_radius} 0 0"/>
     </joint>
 </robot>

Commit message: added imu_link

File: urdf/robot_core.xacro (robot description, xacro)
@@ -15,4 +15,6 @@
     <xacro:property name="sonar_size" value="0.01"/>
     <xacro:property name="sonar_mass" value="0.01"/>
+    <xacro:property name="imu_size" value="0.01"/>
+    <xacro:property name="imu_mass" value="0.01"/>
     <material name="white">
         <color rgba="1.0 1.0 1.0 1.0"/>
@@ -26,4 +28,7 @@
     <material name="blue">
         <color rgba="0 1 1 1"/>
+    </material>
+    <material name="red">
+        <color rgba="0.596078431372549 0.0 0.00784313725490196 1.0"/>
     </material>
     <xacro:macro name="wheel" params="prefix y_reflect">
@@ -118,3 +123,25 @@
         <origin xyz="${disc_radius} 0 0"/>
     </joint>
+    <link name="imu_link">
+        <xacro:box_inertial mass="${imu_mass}" x="${imu_size}" y="${imu_size}" z="${imu_size}"/>
+        <visual>
+            <origin xyz="0 0 0" rpy="0 0 0"/>
+            <geometry>
+                <box size="${imu_size} ${imu_size} ${imu_size}"/>
+            </geometry>
+            <material name="red"/>
+        </visual>
+        <collision>
+            <origin xyz="0 0 0" rpy="0 0 0"/>
+            <geometry>
+                <box size="${imu_size} ${imu_size} ${imu_size}"/>
+            </geometry>
+        </collision>
+    </link>
+    <joint name="imu_joint" type="fixed">
+        <origin xyz="0 0 0" rpy="0 0 0"/>
+        <parent link="base_link"/>
+        <child link="imu_link"/>
+        <axis xyz="0 0 0"/>
+    </joint>
 </robot>

Commit message: refactor

File: urdf/robot_core.xacro (robot description, xacro)
@@ -57,4 +57,5 @@
         </joint>
     </xacro:macro>
+    <link name="base_footprint"/>
     <link name="base_link">
         <xacro:cylinder_inertial mass="${disc_mass}" radius="${disc_radius}" length="${disc_height}" rotation="0"/>
@@ -73,5 +74,4 @@
         </collision>
     </link>
-    <link name="base_footprint"/>
     <joint name="base_footprint_joint" type="fixed">
         <parent link="base_link"/>
