Commit message: ros2 control

File: urdf/two_wheels/two_wheels_macro.ros2_control.xacro (robot description, xacro)
@@ -26,91 +26,20 @@
         </xacro:unless>
       </hardware>
-      <joint name="${prefix}joint1">
-        <command_interface name="position">     <!-- Add/Remove interfaces as needed -->
-          <param name="min">-1</param>
-          <param name="max">1</param>
+      <joint name="left_wheel_joint">
+        <command_interface name="velocity">
+          <param name="min">-10</param>
+          <param name="max">10</param>
         </command_interface>
-        <state_interface name="position">
-          <param name="initial_value">0.0</param>
-        </state_interface>
+        <state_interface name="position"/>
         <state_interface name="velocity"/>
-        <state_interface name="acceleration"/>
       </joint>
-      <joint name="${prefix}joint2">
-        <command_interface name="position">     <!-- Add/Remove interfaces as needed -->
-          <param name="min">-1</param>
-          <param name="max">1</param>
+      <joint name="right_wheel_joint">
+        <command_interface name="velocity">
+          <param name="min">-10</param>
+          <param name="max">10</param>
         </command_interface>
-        <state_interface name="position">
-          <param name="initial_value">0.0</param>
-        </state_interface>
+        <state_interface name="position"/>
         <state_interface name="velocity"/>
-        <state_interface name="acceleration"/>
       </joint>
-      <joint name="${prefix}joint3">
-        <command_interface name="position">     <!-- Add/Remove interfaces as needed -->
-          <param name="min">-1</param>
-          <param name="max">1</param>
-        </command_interface>
-        <state_interface name="position">
-          <param name="initial_value">0.0</param>
-        </state_interface>
-        <state_interface name="velocity"/>
-        <state_interface name="acceleration"/>
-      </joint>
-      <joint name="${prefix}joint4">
-        <command_interface name="position">     <!-- Add/Remove interfaces as needed -->
-          <param name="min">-1</param>
-          <param name="max">1</param>
-        </command_interface>
-        <state_interface name="position">
-          <param name="initial_value">0.0</param>
-        </state_interface>
-        <state_interface name="velocity"/>
-        <state_interface name="acceleration"/>
-      </joint>
-      <joint name="${prefix}joint5">
-        <command_interface name="position">     <!-- Add/Remove interfaces as needed -->
-          <param name="min">-1</param>
-          <param name="max">1</param>
-        </command_interface>
-        <state_interface name="position">
-          <param name="initial_value">0.0</param>
-        </state_interface>
-        <state_interface name="velocity"/>
-        <state_interface name="acceleration"/>
-      </joint>
-      <joint name="${prefix}joint6">
-        <command_interface name="position">     <!-- Add/Remove interfaces as needed -->
-          <param name="min">-1</param>
-          <param name="max">1</param>
-        </command_interface>
-        <state_interface name="position">
-          <param name="initial_value">0.0</param>
-        </state_interface>
-        <state_interface name="velocity"/>
-        <state_interface name="acceleration"/>
-      </joint>
-      <sensor name="tcp_fts_sensor">            <!-- Remove/change sensors as needed -->
-        <state_interface name="fx"/>
-        <state_interface name="fy"/>
-        <state_interface name="fz"/>
-        <state_interface name="tx"/>
-        <state_interface name="ty"/>
-        <state_interface name="tz"/>
-        <param name="frame_id">tool0</param>    <!-- Change sensors as needed -->
-        <param name="min_fx">-100</param>
-        <param name="max_fx">100</param>
-        <param name="min_fy">-100</param>
-        <param name="max_fy">100</param>
-        <param name="min_fz">-200</param>
-        <param name="max_fz">200</param>
-        <param name="min_tx">-10</param>
-        <param name="max_tx">10</param>
-        <param name="min_ty">-10</param>
-        <param name="max_ty">10</param>
-        <param name="min_tz">-15</param>
-        <param name="max_tz">15</param>
-      </sensor>
     </ros2_control>
     <xacro:if value="$(arg sim_gazebo_classic)">

Commit message: gazebo diff drive

File: urdf/two_wheels/two_wheels_macro.ros2_control.xacro (robot description, xacro)
@@ -1,49 +1,62 @@
 <?xml version="1.0" encoding="UTF-8"?>
 <robot xmlns:xacro="http://wiki.ros.org/xacro">
-  <xacro:macro name="two_wheels_ros2_control" params="
+    <xacro:macro name="two_wheels_ros2_control" params="
                name
-               use_mock_hardware:=^|false">
-    <ros2_control name="${name}" type="system">
-      <hardware>
-        <xacro:if value="${use_mock_hardware}">
-          <plugin>mock_components/GenericSystem</plugin>
+               use_mock_hardware">
+        <ros2_control name="${name}" type="system">
+            <hardware>
+                <xacro:if value="${use_mock_hardware}">
+                    <plugin>gazebo_ros2_control/GazeboSystem</plugin>
+                </xacro:if>
+                <xacro:unless value="${use_mock_hardware}">
+                    <plugin>two_wheels/ArduinoWheels</plugin>
+                </xacro:unless>
+            </hardware>
+            <joint name="left_wheel_joint">
+                <command_interface name="velocity">
+                    <param name="min">-10</param>
+                    <param name="max">10</param>
+                </command_interface>
+                <state_interface name="position"/>
+                <state_interface name="velocity"/>
+            </joint>
+            <joint name="right_wheel_joint">
+                <command_interface name="velocity">
+                    <param name="min">-10</param>
+                    <param name="max">10</param>
+                </command_interface>
+                <state_interface name="position"/>
+                <state_interface name="velocity"/>
+            </joint>
+        </ros2_control>
+        <xacro:if value="$(arg use_mock_hardware)">
+            <!-- Gazebo plugins -->
+            <!--      <gazebo reference="world">-->
+            <!--      </gazebo>-->
+            <gazebo>
+                <plugin name="gazebo_ros2_control" filename="libgazebo_ros2_control.so">
+                    <robot_param>robot_description</robot_param>
+                    <robot_param_node>robot_state_publisher</robot_param_node>
+                    <parameters>$(find two_wheels)/config/gaz_ros2_ctl_use_sim.yaml</parameters>
+                    <parameters>$(find two_wheels)/config/two_wheels_controllers.yaml</parameters>
+                </plugin>
+                <plugin name="differential_drive_controller" filename="libgazebo_ros_diff_drive.so">
+                    <!-- Wheel Information -->
+                    <left_joint>left_wheel_joint</left_joint>
+                    <right_joint>right_wheel_joint</right_joint>
+                    <wheel_separation>0.09</wheel_separation>
+                    <wheel_diameter>0.033</wheel_diameter>
+                    <!-- Limits -->
+                    <max_wheel_torque>200</max_wheel_torque>
+                    <max_wheel_acceleration>10.0</max_wheel_acceleration>
+                    <!-- Output -->
+                    <odometry_frame>odom</odometry_frame>
+                    <robot_base_frame>base_link</robot_base_frame>
+                    <publish_odom>true</publish_odom>
+                    <publish_odom_tf>true</publish_odom_tf>
+                    <publish_wheel_tf>true</publish_wheel_tf>
+                </plugin>
+            </gazebo>
         </xacro:if>
-<!--        <xacro:if value="${sim_gazebo_classic}">-->
-<!--          <plugin>gazebo_ros2_control/GazeboSystem</plugin>-->
-<!--        </xacro:if>-->
-<!--        <xacro:if value="${sim_gazebo}">-->
-<!--          <plugin>ign_ros2_control/IgnitionSystem</plugin>-->
-<!--        </xacro:if>-->
-        <xacro:unless value="${use_mock_hardware}">
-          <plugin>two_wheels/ArduinoWheels</plugin>
-        </xacro:unless>
-      </hardware>
-      <joint name="left_wheel_joint">
-        <command_interface name="velocity">
-          <param name="min">-10</param>
-          <param name="max">10</param>
-        </command_interface>
-        <state_interface name="position"/>
-        <state_interface name="velocity"/>
-      </joint>
-      <joint name="right_wheel_joint">
-        <command_interface name="velocity">
-          <param name="min">-10</param>
-          <param name="max">10</param>
-        </command_interface>
-        <state_interface name="position"/>
-        <state_interface name="velocity"/>
-      </joint>
-    </ros2_control>
-<!--    <xacro:if value="$(arg sim_gazebo_classic)">-->
-<!--      &lt;!&ndash; Gazebo plugins &ndash;&gt;-->
-<!--      <gazebo reference="world">-->
-<!--      </gazebo>-->
-<!--      <gazebo>-->
-<!--        <plugin filename="libgazebo_ros2_control.so" name="gazebo_ros2_control">-->
-<!--          <parameters>${simulation_controllers}</parameters>-->
-<!--        </plugin>-->
-<!--      </gazebo>-->
-<!--    </xacro:if>-->
-  </xacro:macro>
+    </xacro:macro>
 </robot>

Commit message: gazebo diff drive

File: urdf/two_wheels/two_wheels_macro.ros2_control.xacro (robot description, xacro)
@@ -31,31 +31,5 @@
         </ros2_control>
         <xacro:if value="$(arg use_mock_hardware)">
-            <!-- Gazebo plugins -->
-            <!--      <gazebo reference="world">-->
-            <!--      </gazebo>-->
-            <gazebo>
-                <plugin name="gazebo_ros2_control" filename="libgazebo_ros2_control.so">
-                    <robot_param>robot_description</robot_param>
-                    <robot_param_node>robot_state_publisher</robot_param_node>
-                    <parameters>$(find two_wheels)/config/gaz_ros2_ctl_use_sim.yaml</parameters>
-                    <parameters>$(find two_wheels)/config/two_wheels_controllers.yaml</parameters>
-                </plugin>
-                <plugin name="differential_drive_controller" filename="libgazebo_ros_diff_drive.so">
-                    <!-- Wheel Information -->
-                    <left_joint>left_wheel_joint</left_joint>
-                    <right_joint>right_wheel_joint</right_joint>
-                    <wheel_separation>0.09</wheel_separation>
-                    <wheel_diameter>0.033</wheel_diameter>
-                    <!-- Limits -->
-                    <max_wheel_torque>200</max_wheel_torque>
-                    <max_wheel_acceleration>10.0</max_wheel_acceleration>
-                    <!-- Output -->
-                    <odometry_frame>odom</odometry_frame>
-                    <robot_base_frame>base_link</robot_base_frame>
-                    <publish_odom>true</publish_odom>
-                    <publish_odom_tf>true</publish_odom_tf>
-                    <publish_wheel_tf>true</publish_wheel_tf>
-                </plugin>
-            </gazebo>
+            <xacro:include filename="$(find two_wheels)/urdf/two_wheels/gazebo_control.xacro"/>
         </xacro:if>
     </xacro:macro>

File: urdf/two_wheels/two_wheels_macro.xacro (robot description, xacro)
@@ -8,4 +8,8 @@
     <xacro:property name="wheel_radius" value="0.033"/>
     <xacro:property name="wheel_mass" value="0.01"/>
+    <xacro:property name="caster_wheel_radius" value="${wheel_radius/2}"/>
+    <xacro:property name="caster_wheel_mass" value="0.01"/>
+    <xacro:property name="caster_wheel_offset_x" value="0.06"/>
+    <xacro:property name="caster_wheel_offset_z" value="${caster_wheel_radius}"/>
     <material name="white">
         <color rgba="1.0 1.0 1.0 1.0"/>
@@ -33,18 +37,19 @@
                 </geometry>
             </collision>
-            <xacro:cylinder_inertial mass="${wheel_mass}" radius="${wheel_radius}" length="${wheel_width}" rotation="${pi/2}"/>
+            <xacro:cylinder_inertial mass="${wheel_mass}" radius="${wheel_radius}" length="${wheel_width}"
+                                     rotation="${pi/2}"/>
         </link>
         <joint name="${prefix}_wheel_joint" type="continuous">
             <parent link="base_link"/>
             <child link="${prefix}_wheel"/>
-            <origin xyz="0 ${y_reflect*(disc_radius+(wheel_width/2))} ${wheel_radius}" rpy="0 0 0"/>
+            <origin xyz="0 ${y_reflect*(disc_radius+(wheel_width/2))} 0" rpy="0 0 0"/>
             <axis xyz="0 1 0"/>
         </joint>
     </xacro:macro>
-    <xacro:macro name="two_wheels" >
+    <xacro:macro name="two_wheels">
         <link name="base_link">
             <xacro:cylinder_inertial mass="${disc_mass}" radius="${disc_radius}" length="${disc_height}" rotation="0"/>
             <visual>
-                <origin xyz="0 0 ${wheel_radius}" rpy="0 0 0"/>
+                <origin xyz="0 0 0" rpy="0 0 0"/>
                 <geometry>
                     <cylinder radius="${disc_radius}" length="${disc_height}"/>
@@ -59,11 +64,33 @@
             </collision>
         </link>
-<!--        <joint name="base_joint" type="fixed">-->
-<!--            <parent link="base_footprint"/>-->
-<!--            <child link="base_link"/>-->
-<!--            <origin xyz="0.0 0.0 ${-wheel_radius}" rpy="0 0 0"/>-->
-<!--        </joint>-->
+        <link name="base_footprint"/>
+        <joint name="base_footprint_joint" type="fixed">
+            <parent link="base_link"/>
+            <child link="base_footprint"/>
+            <origin xyz="0 0 0" rpy="0 0 0"/>
+        </joint>
         <xacro:wheel prefix="left" y_reflect="1"/>
         <xacro:wheel prefix="right" y_reflect="-1"/>
+        <link name="caster_wheel">
+            <visual>
+                <geometry>
+                    <sphere radius="${caster_wheel_radius}"/>
+                </geometry>
+                <material name="black"/>
+            </visual>
+            <collision>
+                <geometry>
+                    <sphere radius="${caster_wheel_radius}"/>
+                </geometry>
+            </collision>
+            <xacro:sphere_inertial radius="${caster_wheel_radius}" mass="${caster_wheel_mass}">
+                <origin xyz="0 0 0" rpy="0 0 0"/>
+            </xacro:sphere_inertial>
+        </link>
+        <joint name="caster_wheel_joint" type="fixed">
+            <parent link="base_link"/>
+            <child link="caster_wheel"/>
+            <origin xyz="${caster_wheel_offset_x} 0 -${caster_wheel_offset_z}"/>
+        </joint>
         <gazebo reference="base_link">
             <material>Gazebo/White</material>
@@ -75,4 +102,9 @@
             <material>Gazebo/Black</material>
         </gazebo>
+        <gazebo reference="caster_wheel">
+            <material>Gazebo/White</material>
+            <mu1 value="0.001"/>
+            <mu2 value="0.001"/>
+        </gazebo>
     </xacro:macro>
 </robot>
