Commit message: refactored urdf

File: urdf/two_wheels/two_wheels_macro.xacro (robot description, xacro)
@@ -2,4 +2,5 @@
 <robot xmlns:xacro="http://wiki.ros.org/xacro">
     <xacro:include filename="$(find two_wheels)/urdf/common.xacro"/>
+    <xacro:include filename="$(find two_wheels)/urdf/two_wheels/gazebo.xacro"/>
     <xacro:property name="disc_height" value="0.005"/>
     <xacro:property name="disc_radius" value="0.07"/>
@@ -93,18 +94,4 @@
             <origin xyz="${caster_wheel_offset_x} 0 -${caster_wheel_offset_z}"/>
         </joint>
-        <gazebo reference="base_link">
-            <material>Gazebo/White</material>
-        </gazebo>
-        <gazebo reference="left_wheel">
-            <material>Gazebo/Black</material>
-        </gazebo>
-        <gazebo reference="right_wheel">
-            <material>Gazebo/Black</material>
-        </gazebo>
-        <gazebo reference="caster_wheel">
-            <material>Gazebo/White</material>
-            <mu1 value="0.001"/>
-            <mu2 value="0.001"/>
-        </gazebo>
     </xacro:macro>
 </robot>
