Commit message: added sensor <collision> tag

File: urdf/gazebo/common_inertias.xacro (robot description, xacro)
@@ -20,8 +20,7 @@
     </inertial>
   </xacro:macro>
-  <xacro:macro name="box_inertial" params="x y z mass *origin">
+  <xacro:macro name="box_inertial" params="x y z mass ">
     <inertial>
       <mass value="${mass}" />
-      <xacro:insert_block name="origin" />
       <inertia ixx="${1.0/12 * mass * (y*y + z*z)}" ixy="0.0" ixz="0.0"
         iyy="${1.0/12 * mass * (x*x + z*z)}" iyz="0.0"

File: urdf/robot_core.xacro (robot description, xacro)
@@ -2,5 +2,5 @@
 <robot xmlns:xacro="http://www.ros.org/wiki/xacro">
     <xacro:arg name="is_sim" default="true"/>
-    <xacro:include filename="common.xacro"/>
+    <xacro:include filename="gazebo/common_inertias.xacro"/>
     <xacro:property name="disc_height" value="0.005"/>
     <xacro:property name="disc_radius" value="0.07"/>
@@ -14,4 +14,5 @@
     <xacro:property name="caster_wheel_offset_z" value="${caster_wheel_radius}"/>
     <xacro:property name="sonar_size" value="0.01"/>
+    <xacro:property name="sonar_mass" value="0.01"/>
     <material name="white">
         <color rgba="1.0 1.0 1.0 1.0"/>
@@ -98,4 +99,5 @@
     <link name="sonar_link">
         <visual>
+            <!--            <origin xyz="0 0 0" rpy="${pi/2} 0 0"/>-->
             <geometry>
                 <box size="${sonar_size} ${sonar_size} ${sonar_size}"/>
@@ -103,4 +105,12 @@
             <material name="cyan"/>
         </visual>
+        <collision>
+            <!--            <origin xyz="0 0 0" rpy="${pi/2} 0 0"/>-->
+            <geometry>
+                <box size="${sonar_size} ${sonar_size} ${sonar_size}"/>
+            </geometry>
+            <material name="cyan"/>
+        </collision>
+        <xacro:box_inertial x="${sonar_size}" y="${sonar_size}" z="${sonar_size}" mass="${sonar_mass}"/>
     </link>
     <joint name="sonar_link_joint" type="fixed">
