Commit message: fixed Gazebo color

File: urdf/gazebo/sonar.xacro (robot description, xacro)
@@ -2,5 +2,7 @@
 <robot>
     <gazebo reference="sonar_link">
+        <material>Gazebo/Blue</material>
         <sensor type="ray" name="range_sensor">
+            <visualize>true</visualize>
             <ray>
                 <scan>

File: urdf/robot_core.xacro (robot description, xacro)
@@ -24,5 +24,5 @@
         <color rgba="0 0 0 1"/>
     </material>
-    <material name="cyan">
+    <material name="blue">
         <color rgba="0 1 1 1"/>
     </material>
@@ -103,5 +103,5 @@
                 <box size="${sonar_size} ${sonar_size} ${sonar_size}"/>
             </geometry>
-            <material name="cyan"/>
+            <material name="blue"/>
         </visual>
         <collision>
@@ -110,5 +110,4 @@
                 <box size="${sonar_size} ${sonar_size} ${sonar_size}"/>
             </geometry>
-            <material name="cyan"/>
         </collision>
         <xacro:box_inertial x="${sonar_size}" y="${sonar_size}" z="${sonar_size}" mass="${sonar_mass}"/>

Commit message: fixed sonar sensor self collision

File: urdf/gazebo/sonar.xacro (robot description, xacro)
@@ -16,6 +16,6 @@
                         <samples>10</samples>
                         <resolution>1</resolution>
-                        <min_angle>-0.087</min_angle>
-                        <max_angle>0.087</max_angle>
+                        <min_angle>0</min_angle>
+                        <max_angle>0</max_angle>
                     </vertical>
                 </scan>

File: urdf/robot_core.xacro (robot description, xacro)
@@ -116,5 +116,5 @@
         <parent link="base_link"/>
         <child link="sonar_link"/>
-        <origin xyz="${caster_wheel_offset_x}  0 0"/>
+        <origin xyz="${disc_radius} 0 0.01"/>
     </joint>
 </robot>
