Commit message: bump_go FSM

File: two_wheels_core/urdf/robot.urdf.xacro (robot description, xacro)
@@ -6,5 +6,4 @@
         <xacro:include filename="gazebo/gazebo.xacro"/>
         <xacro:include filename="gazebo/gazebo_control.xacro"/>
-        <xacro:include filename="gazebo/sonar.xacro"/>
         <xacro:include filename="gazebo/imu.xacro"/>
         <xacro:include filename="gazebo/lidar.xacro"/>

File: two_wheels_core/urdf/robot_core.xacro (robot description, xacro)
@@ -12,6 +12,4 @@
     <xacro:property name="caster_wheel_offset_x" value="0.06"/>
     <xacro:property name="caster_wheel_offset_z" value="${caster_wheel_radius}"/>
-    <xacro:property name="sonar_size" value="0.01"/>
-    <xacro:property name="sonar_mass" value="0.01"/>
     <xacro:property name="imu_size" value="0.01"/>
     <xacro:property name="imu_mass" value="0.01"/>
@@ -101,25 +99,4 @@
         <origin xyz="${caster_wheel_offset_x} 0 -${caster_wheel_offset_z}"/>
     </joint>
-    <link name="sonar_link">
-        <visual>
-            <!--            <origin xyz="0 0 0" rpy="${pi/2} 0 0"/>-->
-            <geometry>
-                <box size="${sonar_size} ${sonar_size} ${sonar_size}"/>
-            </geometry>
-            <material name="blue"/>
-        </visual>
-        <collision>
-            <!--            <origin xyz="0 0 0" rpy="${pi/2} 0 0"/>-->
-            <geometry>
-                <box size="${sonar_size} ${sonar_size} ${sonar_size}"/>
-            </geometry>
-        </collision>
-        <xacro:box_inertial x="${sonar_size}" y="${sonar_size}" z="${sonar_size}" mass="${sonar_mass}"/>
-    </link>
-    <joint name="sonar_link_joint" type="fixed">
-        <parent link="base_link"/>
-        <child link="sonar_link"/>
-        <origin xyz="${disc_radius} 0 0"/>
-    </joint>
     <link name="imu_link">
         <xacro:box_inertial mass="${imu_mass}" x="${imu_size}" y="${imu_size}" z="${imu_size}"/>

Commit message: disabled imu & lidar

File: two_wheels_core/urdf/robot.urdf.xacro (robot description, xacro)
@@ -6,6 +6,6 @@
         <xacro:include filename="gazebo/gazebo.xacro"/>
         <xacro:include filename="gazebo/gazebo_control.xacro"/>
-        <xacro:include filename="gazebo/imu.xacro"/>
-        <xacro:include filename="gazebo/lidar.xacro"/>
+        <!--        <xacro:include filename="gazebo/imu.xacro"/>-->
+        <!--        <xacro:include filename="gazebo/lidar.xacro"/>-->
     </xacro:if>
     <xacro:unless value="$(arg is_sim)">

File: two_wheels_core/urdf/robot_core.xacro (robot description, xacro)
@@ -99,52 +99,3 @@
         <origin xyz="${caster_wheel_offset_x} 0 -${caster_wheel_offset_z}"/>
     </joint>
-    <link name="imu_link">
-        <xacro:box_inertial mass="${imu_mass}" x="${imu_size}" y="${imu_size}" z="${imu_size}"/>
-        <visual>
-            <origin xyz="0 0 0" rpy="0 0 0"/>
-            <geometry>
-                <box size="${imu_size} ${imu_size} ${imu_size}"/>
-            </geometry>
-            <material name="red"/>
-        </visual>
-        <collision>
-            <origin xyz="0 0 0" rpy="0 0 0"/>
-            <geometry>
-                <box size="${imu_size} ${imu_size} ${imu_size}"/>
-            </geometry>
-        </collision>
-    </link>
-    <joint name="imu_joint" type="fixed">
-        <origin xyz="0 0 0" rpy="0 0 0"/>
-        <parent link="base_link"/>
-        <child link="imu_link"/>
-        <axis xyz="0 0 0"/>
-    </joint>
-    <link name="lidar_link">
-        <visual>
-            <geometry>
-                <cylinder radius="0.05" length="0.04"/>
-            </geometry>
-            <material name="black"/>
-        </visual>
-        <visual>
-            <origin xyz="0 0 -0.05"/>
-            <geometry>
-                <cylinder radius="0.01" length="0.1"/>
-            </geometry>
-            <material name="black"/>
-        </visual>
-        <collision>
-            <geometry>
-                <cylinder radius="0.05" length="0.04"/>
-            </geometry>
-        </collision>
-        <xacro:cylinder_inertial mass="0.1" radius="0.04" length="0.05" rotation="0"/>
-    </link>
-    <joint name="lidar_joint" type="fixed">
-        <origin xyz="0 0 0" rpy="0 0 0"/>
-        <parent link="base_link"/>
-        <child link="lidar_link"/>
-        <axis xyz="0 0 0"/>
-    </joint>
 </robot>
