Commit message: updated wheels' and joint's names

File: two_wheels_core/urdf/joints.macro.xacro (robot description, xacro)
@@ -2,5 +2,5 @@
 <robot xmlns:xacro="http://www.ros.org/wiki/xacro">
     <xacro:macro name="joints">
-        <joint name="left_wheel_joint">
+        <joint name="front_left_wheel_joint">
             <command_interface name="velocity">
                 <param name="min">-10</param>
@@ -10,5 +10,5 @@
             <state_interface name="position"/>
         </joint>
-        <joint name="right_wheel_joint">
+        <joint name="front_right_wheel_joint">
             <command_interface name="velocity">
                 <param name="min">-10</param>

File: two_wheels_core/urdf/robot_core.xacro (robot description, xacro)
@@ -76,6 +76,6 @@
         <origin xyz="0 0 0" rpy="0 0 0"/>
     </joint>
-    <xacro:wheel prefix="left" y_reflect="1"/>
-    <xacro:wheel prefix="right" y_reflect="-1"/>
+    <xacro:wheel prefix="front_left" y_reflect="1"/>
+    <xacro:wheel prefix="front_right" y_reflect="-1"/>
     <link name="caster_wheel">
         <visual>

Commit message: finally worked using https://github.com/dheena2k2/fusion2urdf-ros2

File: two_wheels_core/urdf/joints.macro.xacro (robot description, xacro)
@@ -18,4 +18,20 @@
             <state_interface name="position"/>
         </joint>
+        <joint name="rear_left_wheel_joint">
+            <command_interface name="velocity">
+                <param name="min">-10</param>
+                <param name="max">10</param>
+            </command_interface>
+            <state_interface name="velocity"/>
+            <state_interface name="position"/>
+        </joint>
+        <joint name="rear_right_wheel_joint">
+            <command_interface name="velocity">
+                <param name="min">-10</param>
+                <param name="max">10</param>
+            </command_interface>
+            <state_interface name="velocity"/>
+            <state_interface name="position"/>
+        </joint>
     </xacro:macro>
 </robot>

File: two_wheels_core/urdf/robot_core.xacro (robot description, xacro)
@@ -1,75 +1,141 @@
 <?xml version="1.0"?>
 <robot xmlns:xacro="http://www.ros.org/wiki/xacro">
-    <xacro:include filename="gazebo/common_inertias.xacro"/>
-    <xacro:property name="disc_height" value="0.005"/>
-    <xacro:property name="disc_radius" value="0.07"/>
-    <xacro:property name="disc_mass" value="0.05"/>
-    <xacro:property name="wheel_width" value="0.025"/>
-    <xacro:property name="wheel_radius" value="0.024"/>
-    <xacro:property name="wheel_mass" value="0.01"/>
-    <xacro:property name="caster_wheel_radius" value="${wheel_radius/2}"/>
-    <xacro:property name="caster_wheel_mass" value="0.01"/>
-    <xacro:property name="caster_wheel_offset_x" value="0.06"/>
-    <xacro:property name="caster_wheel_offset_z" value="${caster_wheel_radius}"/>
-    <xacro:property name="imu_size" value="0.01"/>
-    <xacro:property name="imu_mass" value="0.01"/>
-    <material name="white">
-        <color rgba="1.0 1.0 1.0 1.0"/>
-    </material>
-    <material name="orange">
-        <color rgba="1 0.3 0.1 1"/>
-    </material>
-    <material name="black">
-        <color rgba="0 0 0 1"/>
-    </material>
-    <material name="blue">
-        <color rgba="0 1 1 1"/>
-    </material>
-    <material name="red">
-        <color rgba="0.596078431372549 0.0 0.00784313725490196 1.0"/>
-    </material>
+    <xacro:include filename="$(find two_wheels_core)/urdf/materials.xacro"/>
+    <!--    <xacro:include filename="$(find two_wheels_core)/urdf/two_wheels_core.trans"/>-->
+    <!--    <xacro:include filename="$(find two_wheels_core)/urdf/two_wheels_core.gazebo"/>-->
     <link name="base_link">
-        <xacro:cylinder_inertial mass="${disc_mass}" radius="${disc_radius}" length="${disc_height}" rotation="0"/>
+        <inertial>
+            <origin xyz="0.0 2.3684273442397533e-17 0.025" rpy="0 0 0"/>
+            <mass value="6.028923307511652"/>
+            <inertia ixx="0.02914" iyy="0.013063" izz="0.041801" ixy="0.0" iyz="0.0" ixz="0.0"/>
+        </inertial>
         <visual>
             <origin xyz="0 0 0" rpy="0 0 0"/>
             <geometry>
-                <cylinder radius="${disc_radius}" length="${disc_height}"/>
+                <mesh filename="file://$(find two_wheels_core)/urdf/meshes/base_link.stl"
+                      scale="0.001 0.001 0.001"/>
             </geometry>
-            <material name="white"/>
+            <material name="silver"/>
         </visual>
         <collision>
             <origin xyz="0 0 0" rpy="0 0 0"/>
             <geometry>
-                <cylinder radius="${disc_radius}" length="${disc_height}"/>
+                <mesh filename="file://$(find two_wheels_core)/urdf/meshes/base_link.stl"
+                      scale="0.001 0.001 0.001"/>
             </geometry>
         </collision>
     </link>
-    <xacro:macro name="wheel" params="prefix y_reflect">
-        <link name="${prefix}_wheel">
-            <visual>
-                <origin xyz="0 0 0" rpy="${pi/2} 0 0"/>
-                <geometry>
-                    <cylinder radius="${wheel_radius}" length="${wheel_width}"/>
-                </geometry>
-                <material name="black"/>
-            </visual>
-            <collision>
-                <origin xyz="0 0 0" rpy="${pi/2} 0 0"/>
-                <geometry>
-                    <cylinder radius="${wheel_radius}" length="${wheel_width}"/>
-                </geometry>
-            </collision>
-            <xacro:cylinder_inertial mass="${wheel_mass}" radius="${wheel_radius}" length="${wheel_width}"
-                                     rotation="${pi/2}"/>
-        </link>
-        <joint name="${prefix}_wheel_joint" type="continuous">
-            <parent link="base_link"/>
-            <child link="${prefix}_wheel"/>
-            <origin xyz="0 ${y_reflect*(disc_radius+(wheel_width/2))} 0" rpy="0 0 0"/>
-            <axis xyz="0 1 0"/>
-        </joint>
-    </xacro:macro>
-    <xacro:wheel prefix="front_left" y_reflect="1"/>
-    <xacro:wheel prefix="front_right" y_reflect="-1"/>
+    <link name="rear_left_wheel">
+        <inertial>
+            <origin xyz="-0.012500000000000011 -2.7755575615628914e-17 0.0" rpy="0 0 0"/>
+            <mass value="0.3549714991722238"/>
+            <inertia ixx="0.000102" iyy="7e-05" izz="7e-05" ixy="0.0" iyz="-0.0" ixz="0.0"/>
+        </inertial>
+        <visual>
+            <origin xyz="0.08 0.078 -0.025" rpy="0 0 0"/>
+            <geometry>
+                <mesh filename="file://$(find two_wheels_core)/urdf/meshes/rear_left_wheel.stl"
+                      scale="0.001 0.001 0.001"/>
+            </geometry>
+            <material name="silver"/>
+        </visual>
+        <collision>
+            <origin xyz="0.08 0.078 -0.025" rpy="0 0 0"/>
+            <geometry>
+                <mesh filename="file://$(find two_wheels_core)/urdf/meshes/rear_left_wheel.stl"
+                      scale="0.001 0.001 0.001"/>
+            </geometry>
+        </collision>
+    </link>
+    <joint name="rear_left_wheel_joint" type="continuous">
+        <origin xyz="-0.08 -0.078 0.025" rpy="0 0 0"/>
+        <parent link="base_link"/>
+        <child link="rear_left_wheel"/>
+        <axis xyz="1.0 0.0 0.0"/>
+    </joint>
+    <link name="front_right_wheel">
+        <inertial>
+            <origin xyz="0.012499999999999997 2.7755575615628914e-17 0.0" rpy="0 0 0"/>
+            <mass value="0.3549714991722238"/>
+            <inertia ixx="0.000102" iyy="7e-05" izz="7e-05" ixy="0.0" iyz="0.0" ixz="-0.0"/>
+        </inertial>
+        <visual>
+            <origin xyz="-0.08 -0.078 -0.025" rpy="0 0 0"/>
+            <geometry>
+                <mesh filename="file://$(find two_wheels_core)/urdf/meshes/front_right_wheel.stl"
+                      scale="0.001 0.001 0.001"/>
+            </geometry>
+            <material name="silver"/>
+        </visual>
+        <collision>
+            <origin xyz="-0.08 -0.078 -0.025" rpy="0 0 0"/>
+            <geometry>
+                <mesh filename="file://$(find two_wheels_core)/urdf/meshes/front_right_wheel.stl"
+                      scale="0.001 0.001 0.001"/>
+            </geometry>
+        </collision>
+    </link>
+    <joint name="front_right_wheel_joint" type="continuous">
+        <origin xyz="0.08 0.078 0.025" rpy="0 0 0"/>
+        <parent link="base_link"/>
+        <child link="front_right_wheel"/>
+        <axis xyz="1.0 0.0 0.0"/>
+    </joint>
+    <link name="rear_right_wheel">
+        <inertial>
+            <origin xyz="0.012499999999999997 -2.7755575615628914e-17 0.0" rpy="0 0 0"/>
+            <mass value="0.3549714991722238"/>
+            <inertia ixx="0.000102" iyy="7e-05" izz="7e-05" ixy="0.0" iyz="-0.0" ixz="-0.0"/>
+        </inertial>
+        <visual>
+            <origin xyz="-0.08 0.078 -0.025" rpy="0 0 0"/>
+            <geometry>
+                <mesh filename="file://$(find two_wheels_core)/urdf/meshes/rear_right_wheel.stl"
+                      scale="0.001 0.001 0.001"/>
+            </geometry>
+            <material name="silver"/>
+        </visual>
+        <collision>
+            <origin xyz="-0.08 0.078 -0.025" rpy="0 0 0"/>
+            <geometry>
+                <mesh filename="file://$(find two_wheels_core)/urdf/meshes/rear_right_wheel.stl"
+                      scale="0.001 0.001 0.001"/>
+            </geometry>
+        </collision>
+    </link>
+    <joint name="rear_right_wheel_joint" type="continuous">
+        <origin xyz="0.08 -0.078 0.025" rpy="0 0 0"/>
+        <parent link="base_link"/>
+        <child link="rear_right_wheel"/>
+        <axis xyz="1.0 0.0 0.0"/>
+    </joint>
+    <link name="front_left_wheel">
+        <inertial>
+            <origin xyz="-0.012500000000000011 2.7755575615628914e-17 0.0" rpy="0 0 0"/>
+            <mass value="0.3549714991722238"/>
+            <inertia ixx="0.000102" iyy="7e-05" izz="7e-05" ixy="-0.0" iyz="0.0" ixz="0.0"/>
+        </inertial>
+        <visual>
+            <origin xyz="0.08 -0.078 -0.025" rpy="0 0 0"/>
+            <geometry>
+                <mesh filename="file://$(find two_wheels_core)/urdf/meshes/front_left_wheel.stl"
+                      scale="0.001 0.001 0.001"/>
+            </geometry>
+            <material name="silver"/>
+        </visual>
+        <collision>
+            <origin xyz="0.08 -0.078 -0.025" rpy="0 0 0"/>
+            <geometry>
+                <mesh filename="file://$(find two_wheels_core)/urdf/meshes/front_left_wheel.stl"
+                      scale="0.001 0.001 0.001"/>
+            </geometry>
+        </collision>
+    </link>
+    <joint name="front_left_wheel_joint" type="continuous">
+        <origin xyz="-0.08 0.078 0.025" rpy="0 0 0"/>
+        <parent link="base_link"/>
+        <child link="front_left_wheel"/>
+        <axis xyz="-1.0 0.0 0.0"/>
+    </joint>
     <link name="base_footprint"/>
     <joint name="base_footprint_joint" type="fixed">
