Commit message: removed caster wheel

File: two_wheels_core/urdf/robot_core.xacro (robot description, xacro)
@@ -29,4 +29,20 @@
         <color rgba="0.596078431372549 0.0 0.00784313725490196 1.0"/>
     </material>
+    <link name="base_link">
+        <xacro:cylinder_inertial mass="${disc_mass}" radius="${disc_radius}" length="${disc_height}" rotation="0"/>
+        <visual>
+            <origin xyz="0 0 0" rpy="0 0 0"/>
+            <geometry>
+                <cylinder radius="${disc_radius}" length="${disc_height}"/>
+            </geometry>
+            <material name="white"/>
+        </visual>
+        <collision>
+            <origin xyz="0 0 0" rpy="0 0 0"/>
+            <geometry>
+                <cylinder radius="${disc_radius}" length="${disc_height}"/>
+            </geometry>
+        </collision>
+    </link>
     <xacro:macro name="wheel" params="prefix y_reflect">
         <link name="${prefix}_wheel">
@@ -54,21 +70,7 @@
         </joint>
     </xacro:macro>
+    <xacro:wheel prefix="front_left" y_reflect="1"/>
+    <xacro:wheel prefix="front_right" y_reflect="-1"/>
     <link name="base_footprint"/>
-    <link name="base_link">
-        <xacro:cylinder_inertial mass="${disc_mass}" radius="${disc_radius}" length="${disc_height}" rotation="0"/>
-        <visual>
-            <origin xyz="0 0 0" rpy="0 0 0"/>
-            <geometry>
-                <cylinder radius="${disc_radius}" length="${disc_height}"/>
-            </geometry>
-            <material name="white"/>
-        </visual>
-        <collision>
-            <origin xyz="0 0 0" rpy="0 0 0"/>
-            <geometry>
-                <cylinder radius="${disc_radius}" length="${disc_height}"/>
-            </geometry>
-        </collision>
-    </link>
     <joint name="base_footprint_joint" type="fixed">
         <parent link="base_link"/>
@@ -76,26 +78,3 @@
         <origin xyz="0 0 0" rpy="0 0 0"/>
     </joint>
-    <xacro:wheel prefix="front_left" y_reflect="1"/>
-    <xacro:wheel prefix="front_right" y_reflect="-1"/>
-    <link name="caster_wheel">
-        <visual>
-            <geometry>
-                <sphere radius="${caster_wheel_radius}"/>
-            </geometry>
-            <material name="black"/>
-        </visual>
-        <collision>
-            <geometry>
-                <sphere radius="${caster_wheel_radius}"/>
-            </geometry>
-        </collision>
-        <xacro:sphere_inertial radius="${caster_wheel_radius}" mass="${caster_wheel_mass}">
-            <origin xyz="0 0 0" rpy="0 0 0"/>
-        </xacro:sphere_inertial>
-    </link>
-    <joint name="caster_wheel_joint" type="fixed">
-        <parent link="base_link"/>
-        <child link="caster_wheel"/>
-        <origin xyz="${caster_wheel_offset_x} 0 -${caster_wheel_offset_z}"/>
-    </joint>
 </robot>

Commit message: changed wheel_radius to 0.024

File: two_wheels_core/urdf/robot_core.xacro (robot description, xacro)
@@ -6,5 +6,5 @@
     <xacro:property name="disc_mass" value="0.05"/>
     <xacro:property name="wheel_width" value="0.025"/>
-    <xacro:property name="wheel_radius" value="0.033"/>
+    <xacro:property name="wheel_radius" value="0.024"/>
     <xacro:property name="wheel_mass" value="0.01"/>
     <xacro:property name="caster_wheel_radius" value="${wheel_radius/2}"/>

Commit message: 4 wheel drive working!

File: two_wheels_core/urdf/robot_core.xacro (robot description, xacro)
@@ -114,5 +114,5 @@
         <parent link="base_link"/>
         <child link="front_left_wheel"/>
-        <axis xyz="0.0 -1.0 0.0"/>
+        <axis xyz="0.0 1.0 0.0"/>
     </joint>
     <joint name="rear_left_wheel_joint" type="continuous">
@@ -120,5 +120,5 @@
         <parent link="base_link"/>
         <child link="rear_left_wheel"/>
-        <axis xyz="0.0 -1.0 0.0"/>
+        <axis xyz="0.0 1.0 0.0"/>
     </joint>
     <joint name="rear_right_wheel_joint" type="continuous">
@@ -126,5 +126,5 @@
         <parent link="base_link"/>
         <child link="rear_right_wheel"/>
-        <axis xyz="-0.0 1.0 -0.0"/>
+        <axis xyz="0.0 1.0 0.0"/>
     </joint>
     <joint name="front_right_wheel_joint" type="continuous">
@@ -132,5 +132,5 @@
         <parent link="base_link"/>
         <child link="front_right_wheel"/>
-        <axis xyz="0.0 1.0 -0.0"/>
+        <axis xyz="0.0 1.0 0.0"/>
     </joint>
     <link name="base_footprint"/>

Commit message: fixed lidar_link.stl path

File: two_wheels_core/urdf/robot_core.xacro (robot description, xacro)
@@ -143,5 +143,5 @@
             <origin xyz="-0.11007 -3.2e-05 -0.028463" rpy="0 0 0"/>
             <geometry>
-                <mesh filename="file://$(find two_wheels_core_description)/meshes/lidar_link.stl"
+                <mesh filename="file://$(find two_wheels_core)/urdf/meshes/lidar_link.stl"
                       scale="0.001 0.001 0.001"/>
             </geometry>
@@ -151,5 +151,5 @@
             <origin xyz="-0.11007 -3.2e-05 -0.028463" rpy="0 0 0"/>
             <geometry>
-                <mesh filename="file://$(find two_wheels_core_description)/meshes/lidar_link.stl"
+                <mesh filename="file://$(find two_wheels_core)/urdf/meshes/lidar_link.stl"
                       scale="0.001 0.001 0.001"/>
             </geometry>

Commit message: updated wheels' names

File: two_wheels_core/urdf/robot_core.xacro (robot description, xacro)
@@ -22,5 +22,5 @@
         </collision>
     </link>
-    <link name="front_left_wheel">
+    <link name="rear_right_wheel">
         <inertial>
             <origin xyz="1.625960121487413e-06 -0.03356595189466297 -1.9609319341917786e-09" rpy="0 0 0"/>
@@ -31,4 +31,48 @@
             <origin xyz="0.077933 0.059968 -0.023743" rpy="0 0 0"/>
             <geometry>
+                <mesh filename="file://$(find two_wheels_core)/urdf/meshes/rear_right_wheel.stl"
+                      scale="0.001 0.001 0.001"/>
+            </geometry>
+            <material name="black"/>
+        </visual>
+        <collision>
+            <origin xyz="0.077933 0.059968 -0.023743" rpy="0 0 0"/>
+            <geometry>
+                <mesh filename="file://$(find two_wheels_core)/urdf/meshes/rear_right_wheel.stl"
+                      scale="0.001 0.001 0.001"/>
+            </geometry>
+        </collision>
+    </link>
+    <link name="front_right_wheel">
+        <inertial>
+            <origin xyz="1.3407781088436987e-06 -0.03356595189466117 -1.9609318023527944e-09" rpy="0 0 0"/>
+            <mass value="0.2182048906279955"/>
+            <inertia ixx="3.8e-05" iyy="4.8e-05" izz="3.8e-05" ixy="0.0" iyz="0.0" ixz="0.0"/>
+        </inertial>
+        <visual>
+            <origin xyz="-0.077933 0.059968 -0.023743" rpy="0 0 0"/>
+            <geometry>
+                <mesh filename="file://$(find two_wheels_core)/urdf/meshes/front_right_wheel.stl"
+                      scale="0.001 0.001 0.001"/>
+            </geometry>
+            <material name="black"/>
+        </visual>
+        <collision>
+            <origin xyz="-0.077933 0.059968 -0.023743" rpy="0 0 0"/>
+            <geometry>
+                <mesh filename="file://$(find two_wheels_core)/urdf/meshes/front_right_wheel.stl"
+                      scale="0.001 0.001 0.001"/>
+            </geometry>
+        </collision>
+    </link>
+    <link name="front_left_wheel">
+        <inertial>
+            <origin xyz="1.4899030495729715e-06 0.03356602362407317 3.1974513525767634e-07" rpy="0 0 0"/>
+            <mass value="0.2182048906279955"/>
+            <inertia ixx="3.8e-05" iyy="4.8e-05" izz="3.8e-05" ixy="-0.0" iyz="0.0" ixz="-0.0"/>
+        </inertial>
+        <visual>
+            <origin xyz="-0.077931 -0.060032 -0.023742" rpy="0 0 0"/>
+            <geometry>
                 <mesh filename="file://$(find two_wheels_core)/urdf/meshes/front_left_wheel.stl"
                       scale="0.001 0.001 0.001"/>
@@ -37,5 +81,5 @@
         </visual>
         <collision>
-            <origin xyz="0.077933 0.059968 -0.023743" rpy="0 0 0"/>
+            <origin xyz="-0.077931 -0.060032 -0.023742" rpy="0 0 0"/>
             <geometry>
                 <mesh filename="file://$(find two_wheels_core)/urdf/meshes/front_left_wheel.stl"
@@ -46,10 +90,10 @@
     <link name="rear_left_wheel">
         <inertial>
-            <origin xyz="1.3407781088436987e-06 -0.03356595189466117 -1.9609318023527944e-09" rpy="0 0 0"/>
+            <origin xyz="-1.489903047255381e-06 0.033566023624073626 8.554326641832533e-08" rpy="0 0 0"/>
             <mass value="0.2182048906279955"/>
-            <inertia ixx="3.8e-05" iyy="4.8e-05" izz="3.8e-05" ixy="0.0" iyz="0.0" ixz="0.0"/>
+            <inertia ixx="3.8e-05" iyy="4.8e-05" izz="3.8e-05" ixy="0.0" iyz="-0.0" ixz="-0.0"/>
         </inertial>
         <visual>
-            <origin xyz="-0.077933 0.059968 -0.023743" rpy="0 0 0"/>
+            <origin xyz="0.077931 -0.060032 -0.023742" rpy="0 0 0"/>
             <geometry>
                 <mesh filename="file://$(find two_wheels_core)/urdf/meshes/rear_left_wheel.stl"
@@ -59,5 +103,5 @@
         </visual>
         <collision>
-            <origin xyz="-0.077933 0.059968 -0.023743" rpy="0 0 0"/>
+            <origin xyz="0.077931 -0.060032 -0.023742" rpy="0 0 0"/>
             <geometry>
                 <mesh filename="file://$(find two_wheels_core)/urdf/meshes/rear_left_wheel.stl"
@@ -66,50 +110,18 @@
         </collision>
     </link>
-    <link name="rear_right_wheel">
-        <inertial>
-            <origin xyz="1.4899030495729715e-06 0.03356602362407317 3.1974513525767634e-07" rpy="0 0 0"/>
-            <mass value="0.2182048906279955"/>
-            <inertia ixx="3.8e-05" iyy="4.8e-05" izz="3.8e-05" ixy="-0.0" iyz="0.0" ixz="-0.0"/>
-        </inertial>
-        <visual>
-            <origin xyz="-0.077931 -0.060032 -0.023742" rpy="0 0 0"/>
-            <geometry>
-                <mesh filename="file://$(find two_wheels_core)/urdf/meshes/rear_right_wheel.stl"
-                      scale="0.001 0.001 0.001"/>
-            </geometry>
-            <material name="black"/>
-        </visual>
-        <collision>
-            <origin xyz="-0.077931 -0.060032 -0.023742" rpy="0 0 0"/>
-            <geometry>
-                <mesh filename="file://$(find two_wheels_core)/urdf/meshes/rear_right_wheel.stl"
-                      scale="0.001 0.001 0.001"/>
-            </geometry>
-        </collision>
-    </link>
-    <link name="front_right_wheel">
-        <inertial>
-            <origin xyz="-1.489903047255381e-06 0.033566023624073626 8.554326641832533e-08" rpy="0 0 0"/>
-            <mass value="0.2182048906279955"/>
-            <inertia ixx="3.8e-05" iyy="4.8e-05" izz="3.8e-05" ixy="0.0" iyz="-0.0" ixz="-0.0"/>
-        </inertial>
-        <visual>
-            <origin xyz="0.077931 -0.060032 -0.023742" rpy="0 0 0"/>
-            <geometry>
-                <mesh filename="file://$(find two_wheels_core)/urdf/meshes/front_right_wheel.stl"
-                      scale="0.001 0.001 0.001"/>
-            </geometry>
-            <material name="black"/>
-        </visual>
-        <collision>
-            <origin xyz="0.077931 -0.060032 -0.023742" rpy="0 0 0"/>
-            <geometry>
-                <mesh filename="file://$(find two_wheels_core)/urdf/meshes/front_right_wheel.stl"
-                      scale="0.001 0.001 0.001"/>
-            </geometry>
-        </collision>
-    </link>
+    <joint name="rear_right_wheel_joint" type="continuous">
+        <origin xyz="-0.077933 -0.059968 0.023743" rpy="0 0 0"/>
+        <parent link="base_link"/>
+        <child link="rear_right_wheel"/>
+        <axis xyz="0.0 1.0 0.0"/>
+    </joint>
+    <joint name="front_right_wheel_joint" type="continuous">
+        <origin xyz="0.077933 -0.059968 0.023743" rpy="0 0 0"/>
+        <parent link="base_link"/>
+        <child link="front_right_wheel"/>
+        <axis xyz="0.0 1.0 0.0"/>
+    </joint>
     <joint name="front_left_wheel_joint" type="continuous">
-        <origin xyz="-0.077933 -0.059968 0.023743" rpy="0 0 0"/>
+        <origin xyz="0.077931 0.060032 0.023742" rpy="0 0 0"/>
         <parent link="base_link"/>
         <child link="front_left_wheel"/>
@@ -117,19 +129,7 @@
     </joint>
     <joint name="rear_left_wheel_joint" type="continuous">
-        <origin xyz="0.077933 -0.059968 0.023743" rpy="0 0 0"/>
+        <origin xyz="-0.077931 0.060032 0.023742" rpy="0 0 0"/>
         <parent link="base_link"/>
         <child link="rear_left_wheel"/>
-        <axis xyz="0.0 1.0 0.0"/>
-    </joint>
-    <joint name="rear_right_wheel_joint" type="continuous">
-        <origin xyz="0.077931 0.060032 0.023742" rpy="0 0 0"/>
-        <parent link="base_link"/>
-        <child link="rear_right_wheel"/>
-        <axis xyz="0.0 1.0 0.0"/>
-    </joint>
-    <joint name="front_right_wheel_joint" type="continuous">
-        <origin xyz="-0.077931 0.060032 0.023742" rpy="0 0 0"/>
-        <parent link="base_link"/>
-        <child link="front_right_wheel"/>
         <axis xyz="0.0 1.0 0.0"/>
     </joint>
