Commit message: 4 wheel drive from fusion 360

File: two_wheels_core/urdf/gazebo/gazebo.xacro (robot description, xacro)
@@ -1,35 +1,35 @@
 <?xml version="1.0" encoding="UTF-8"?>
-<robot>
+<robot xmlns:xacro="http://www.ros.org/wiki/xacro">
+    <xacro:property name="body_color" value="Gazebo/Silver"/>
     <gazebo reference="base_link">
-        <material>Gazebo/White</material>
+        <material>${body_color}</material>
+        <mu1>0.2</mu1>
+        <mu2>0.2</mu2>
+        <self_collide>true</self_collide>
+        <gravity>true</gravity>
     </gazebo>
-    <gazebo reference="left_wheel">
-        <material>Gazebo/Black</material>
-        <mu1>1000000000000000.0</mu1>
-        <mu2>1000000000000000.0</mu2>
-        <kp>1000000000000.0</kp>
-        <kd>10.0</kd>
-        <minDepth>0.001</minDepth>
-        <maxVel>0.1</maxVel>
-        <fdir1>1 0 0</fdir1>
+    <gazebo reference="front_left_wheel_1">
+        <material>${body_color}</material>
+        <mu1>0.2</mu1>
+        <mu2>0.2</mu2>
+        <self_collide>true</self_collide>
     </gazebo>
-    <gazebo reference="right_wheel">
-        <material>Gazebo/Black</material>
-        <mu1>1000000000000000.0</mu1>
-        <mu2>1000000000000000.0</mu2>
-        <kp>1000000000000.0</kp>
-        <kd>10.0</kd>
-        <minDepth>0.001</minDepth>
-        <maxVel>0.1</maxVel>
-        <fdir1>1 0 0</fdir1>
+    <gazebo reference="rear_left_wheel_1">
+        <material>${body_color}</material>
+        <mu1>0.2</mu1>
+        <mu2>0.2</mu2>
+        <self_collide>true</self_collide>
     </gazebo>
-    <gazebo reference="caster_wheel">
-        <material>Gazebo/White</material>
-        <mu1>0.1</mu1>
-        <mu2>0.1</mu2>
-        <kp>1000000.0</kp>
-        <kd>100.0</kd>
-        <minDepth>0.001</minDepth>
-        <maxVel>1.0</maxVel>
+    <gazebo reference="rear_right_wheel_1">
+        <material>${body_color}</material>
+        <mu1>0.2</mu1>
+        <mu2>0.2</mu2>
+        <self_collide>true</self_collide>
+    </gazebo>
+    <gazebo reference="front_right_wheel_1">
+        <material>${body_color}</material>
+        <mu1>0.2</mu1>
+        <mu2>0.2</mu2>
+        <self_collide>true</self_collide>
     </gazebo>
 </robot>

File: two_wheels_core/urdf/robot_core.xacro (robot description, xacro)
@@ -2,17 +2,14 @@
 <robot xmlns:xacro="http://www.ros.org/wiki/xacro">
     <xacro:include filename="$(find two_wheels_core)/urdf/materials.xacro"/>
-    <!--    <xacro:include filename="$(find two_wheels_core)/urdf/two_wheels_core.trans"/>-->
-    <!--    <xacro:include filename="$(find two_wheels_core)/urdf/two_wheels_core.gazebo"/>-->
     <link name="base_link">
         <inertial>
-            <origin xyz="0.0 2.3684273442397533e-17 0.025" rpy="0 0 0"/>
-            <mass value="6.028923307511652"/>
-            <inertia ixx="0.02914" iyy="0.013063" izz="0.041801" ixy="0.0" iyz="0.0" ixz="0.0"/>
+            <origin xyz="7.136447167432144e-05 3.453515765351803e-05 0.024408245184796683" rpy="0 0 0"/>
+            <mass value="1.000593039456424"/>
+            <inertia ixx="0.003708" iyy="0.007317" izz="0.010943" ixy="-0.0" iyz="-0.0" ixz="-0.0"/>
         </inertial>
         <visual>
             <origin xyz="0 0 0" rpy="0 0 0"/>
             <geometry>
-                <mesh filename="file://$(find two_wheels_core)/urdf/meshes/base_link.stl"
-                      scale="0.001 0.001 0.001"/>
+                <mesh filename="file://$(find two_wheels_core)/urdf/meshes/base_link.stl" scale="0.001 0.001 0.001"/>
             </geometry>
             <material name="silver"/>
@@ -21,5 +18,26 @@
             <origin xyz="0 0 0" rpy="0 0 0"/>
             <geometry>
-                <mesh filename="file://$(find two_wheels_core)/urdf/meshes/base_link.stl"
+                <mesh filename="file://$(find two_wheels_core)/urdf/meshes/base_link.stl" scale="0.001 0.001 0.001"/>
+            </geometry>
+        </collision>
+    </link>
+    <link name="front_left_wheel">
+        <inertial>
+            <origin xyz="1.625960121487413e-06 -0.03356595189466297 -1.9609319341917786e-09" rpy="0 0 0"/>
+            <mass value="0.21820489062799583"/>
+            <inertia ixx="3.8e-05" iyy="4.8e-05" izz="3.8e-05" ixy="0.0" iyz="0.0" ixz="0.0"/>
+        </inertial>
+        <visual>
+            <origin xyz="0.077933 0.059968 -0.023743" rpy="0 0 0"/>
+            <geometry>
+                <mesh filename="file://$(find two_wheels_core)/urdf/meshes/front_left_wheel.stl"
+                      scale="0.001 0.001 0.001"/>
+            </geometry>
+            <material name="silver"/>
+        </visual>
+        <collision>
+            <origin xyz="0.077933 0.059968 -0.023743" rpy="0 0 0"/>
+            <geometry>
+                <mesh filename="file://$(find two_wheels_core)/urdf/meshes/front_left_wheel.stl"
                       scale="0.001 0.001 0.001"/>
             </geometry>
@@ -28,10 +46,10 @@
     <link name="rear_left_wheel">
         <inertial>
-            <origin xyz="-0.012500000000000011 -2.7755575615628914e-17 0.0" rpy="0 0 0"/>
-            <mass value="0.3549714991722238"/>
-            <inertia ixx="0.000102" iyy="7e-05" izz="7e-05" ixy="0.0" iyz="-0.0" ixz="0.0"/>
+            <origin xyz="1.3407781088436987e-06 -0.03356595189466117 -1.9609318023527944e-09" rpy="0 0 0"/>
+            <mass value="0.2182048906279955"/>
+            <inertia ixx="3.8e-05" iyy="4.8e-05" izz="3.8e-05" ixy="0.0" iyz="0.0" ixz="0.0"/>
         </inertial>
         <visual>
-            <origin xyz="0.08 0.078 -0.025" rpy="0 0 0"/>
+            <origin xyz="-0.077933 0.059968 -0.023743" rpy="0 0 0"/>
             <geometry>
                 <mesh filename="file://$(find two_wheels_core)/urdf/meshes/rear_left_wheel.stl"
@@ -41,5 +59,5 @@
         </visual>
         <collision>
-            <origin xyz="0.08 0.078 -0.025" rpy="0 0 0"/>
+            <origin xyz="-0.077933 0.059968 -0.023743" rpy="0 0 0"/>
             <geometry>
                 <mesh filename="file://$(find two_wheels_core)/urdf/meshes/rear_left_wheel.stl"
@@ -48,18 +66,34 @@
         </collision>
     </link>
-    <joint name="rear_left_wheel_joint" type="continuous">
-        <origin xyz="-0.08 -0.078 0.025" rpy="0 0 0"/>
-        <parent link="base_link"/>
-        <child link="rear_left_wheel"/>
-        <axis xyz="1.0 0.0 0.0"/>
-    </joint>
+    <link name="rear_right_wheel">
+        <inertial>
+            <origin xyz="1.4899030495729715e-06 0.03356602362407317 3.1974513525767634e-07" rpy="0 0 0"/>
+            <mass value="0.2182048906279955"/>
+            <inertia ixx="3.8e-05" iyy="4.8e-05" izz="3.8e-05" ixy="-0.0" iyz="0.0" ixz="-0.0"/>
+        </inertial>
+        <visual>
+            <origin xyz="-0.077931 -0.060032 -0.023742" rpy="0 0 0"/>
+            <geometry>
+                <mesh filename="file://$(find two_wheels_core)/urdf/meshes/rear_right_wheel.stl"
+                      scale="0.001 0.001 0.001"/>
+            </geometry>
+            <material name="silver"/>
+        </visual>
+        <collision>
+            <origin xyz="-0.077931 -0.060032 -0.023742" rpy="0 0 0"/>
+            <geometry>
+                <mesh filename="file://$(find two_wheels_core)/urdf/meshes/rear_right_wheel.stl"
+                      scale="0.001 0.001 0.001"/>
+            </geometry>
+        </collision>
+    </link>
     <link name="front_right_wheel">
         <inertial>
-            <origin xyz="0.012499999999999997 2.7755575615628914e-17 0.0" rpy="0 0 0"/>
-            <mass value="0.3549714991722238"/>
-            <inertia ixx="0.000102" iyy="7e-05" izz="7e-05" ixy="0.0" iyz="0.0" ixz="-0.0"/>
+            <origin xyz="-1.489903047255381e-06 0.033566023624073626 8.554326641832533e-08" rpy="0 0 0"/>
+            <mass value="0.2182048906279955"/>
+            <inertia ixx="3.8e-05" iyy="4.8e-05" izz="3.8e-05" ixy="0.0" iyz="-0.0" ixz="-0.0"/>
         </inertial>
         <visual>
-            <origin xyz="-0.08 -0.078 -0.025" rpy="0 0 0"/>
+            <origin xyz="0.077931 -0.060032 -0.023742" rpy="0 0 0"/>
             <geometry>
                 <mesh filename="file://$(find two_wheels_core)/urdf/meshes/front_right_wheel.stl"
@@ -69,5 +103,5 @@
         </visual>
         <collision>
-            <origin xyz="-0.08 -0.078 -0.025" rpy="0 0 0"/>
+            <origin xyz="0.077931 -0.060032 -0.023742" rpy="0 0 0"/>
             <geometry>
                 <mesh filename="file://$(find two_wheels_core)/urdf/meshes/front_right_wheel.stl"
@@ -76,65 +110,27 @@
         </collision>
     </link>
+    <joint name="front_left_wheel_joint" type="continuous">
+        <origin xyz="-0.077933 -0.059968 0.023743" rpy="0 0 0"/>
+        <parent link="base_link"/>
+        <child link="front_left_wheel"/>
+        <axis xyz="0.0 -1.0 0.0"/>
+    </joint>
+    <joint name="rear_left_wheel_joint" type="continuous">
+        <origin xyz="0.077933 -0.059968 0.023743" rpy="0 0 0"/>
+        <parent link="base_link"/>
+        <child link="rear_left_wheel"/>
+        <axis xyz="0.0 -1.0 0.0"/>
+    </joint>
+    <joint name="rear_right_wheel_joint" type="continuous">
+        <origin xyz="0.077931 0.060032 0.023742" rpy="0 0 0"/>
+        <parent link="base_link"/>
+        <child link="rear_right_wheel"/>
+        <axis xyz="-0.0 1.0 -0.0"/>
+    </joint>
     <joint name="front_right_wheel_joint" type="continuous">
-        <origin xyz="0.08 0.078 0.025" rpy="0 0 0"/>
+        <origin xyz="-0.077931 0.060032 0.023742" rpy="0 0 0"/>
         <parent link="base_link"/>
         <child link="front_right_wheel"/>
-        <axis xyz="1.0 0.0 0.0"/>
-    </joint>
-    <link name="rear_right_wheel">
-        <inertial>
-            <origin xyz="0.012499999999999997 -2.7755575615628914e-17 0.0" rpy="0 0 0"/>
-            <mass value="0.3549714991722238"/>
-            <inertia ixx="0.000102" iyy="7e-05" izz="7e-05" ixy="0.0" iyz="-0.0" ixz="-0.0"/>
-        </inertial>
-        <visual>
-            <origin xyz="-0.08 0.078 -0.025" rpy="0 0 0"/>
-            <geometry>
-                <mesh filename="file://$(find two_wheels_core)/urdf/meshes/rear_right_wheel.stl"
-                      scale="0.001 0.001 0.001"/>
-            </geometry>
-            <material name="silver"/>
-        </visual>
-        <collision>
-            <origin xyz="-0.08 0.078 -0.025" rpy="0 0 0"/>
-            <geometry>
-                <mesh filename="file://$(find two_wheels_core)/urdf/meshes/rear_right_wheel.stl"
-                      scale="0.001 0.001 0.001"/>
-            </geometry>
-        </collision>
-    </link>
-    <joint name="rear_right_wheel_joint" type="continuous">
-        <origin xyz="0.08 -0.078 0.025" rpy="0 0 0"/>
-        <parent link="base_link"/>
-        <child link="rear_right_wheel"/>
-        <axis xyz="1.0 0.0 0.0"/>
-    </joint>
-    <link name="front_left_wheel">
-        <inertial>
-            <origin xyz="-0.012500000000000011 2.7755575615628914e-17 0.0" rpy="0 0 0"/>
-            <mass value="0.3549714991722238"/>
-            <inertia ixx="0.000102" iyy="7e-05" izz="7e-05" ixy="-0.0" iyz="0.0" ixz="0.0"/>
-        </inertial>
-        <visual>
-            <origin xyz="0.08 -0.078 -0.025" rpy="0 0 0"/>
-            <geometry>
-                <mesh filename="file://$(find two_wheels_core)/urdf/meshes/front_left_wheel.stl"
-                      scale="0.001 0.001 0.001"/>
-            </geometry>
-            <material name="silver"/>
-        </visual>
-        <collision>
-            <origin xyz="0.08 -0.078 -0.025" rpy="0 0 0"/>
-            <geometry>
-                <mesh filename="file://$(find two_wheels_core)/urdf/meshes/front_left_wheel.stl"
-                      scale="0.001 0.001 0.001"/>
-            </geometry>
-        </collision>
-    </link>
-    <joint name="front_left_wheel_joint" type="continuous">
-        <origin xyz="-0.08 0.078 0.025" rpy="0 0 0"/>
-        <parent link="base_link"/>
-        <child link="front_left_wheel"/>
-        <axis xyz="-1.0 0.0 0.0"/>
+        <axis xyz="0.0 1.0 -0.0"/>
     </joint>
     <link name="base_footprint"/>

Commit message: lidar_link

File: two_wheels_core/urdf/gazebo/gazebo.xacro (robot description, xacro)
@@ -9,5 +9,5 @@
         <gravity>true</gravity>
     </gazebo>
-    <gazebo reference="front_left_wheel_1">
+    <gazebo reference="front_left_wheel">
         <material>${body_color}</material>
         <mu1>0.2</mu1>
@@ -15,5 +15,5 @@
         <self_collide>true</self_collide>
     </gazebo>
-    <gazebo reference="rear_left_wheel_1">
+    <gazebo reference="rear_left_wheel">
         <material>${body_color}</material>
         <mu1>0.2</mu1>
@@ -21,5 +21,5 @@
         <self_collide>true</self_collide>
     </gazebo>
-    <gazebo reference="rear_right_wheel_1">
+    <gazebo reference="rear_right_wheel">
         <material>${body_color}</material>
         <mu1>0.2</mu1>
@@ -27,5 +27,11 @@
         <self_collide>true</self_collide>
     </gazebo>
-    <gazebo reference="front_right_wheel_1">
+    <gazebo reference="front_right_wheel">
+        <material>${body_color}</material>
+        <mu1>0.2</mu1>
+        <mu2>0.2</mu2>
+        <self_collide>true</self_collide>
+    </gazebo>
+    <gazebo reference="lidar_link">
         <material>${body_color}</material>
         <mu1>0.2</mu1>

File: two_wheels_core/urdf/robot.xacro (robot description, xacro)
@@ -7,5 +7,5 @@
         <xacro:include filename="gazebo/gazebo_control.xacro"/>
         <!--        <xacro:include filename="gazebo/imu.xacro"/>-->
-        <!--        <xacro:include filename="gazebo/lidar.xacro"/>-->
+        <xacro:include filename="gazebo/lidar.xacro"/>
     </xacro:if>
     <xacro:unless value="$(arg is_sim)">

File: two_wheels_core/urdf/robot_core.xacro (robot description, xacro)
@@ -134,4 +134,31 @@
         <axis xyz="0.0 1.0 0.0"/>
     </joint>
+    <link name="lidar_link">
+        <inertial>
+            <origin xyz="-0.00011530732368342234 3.558559248059221e-06 0.017945212221916012" rpy="0 0 0"/>
+            <mass value="0.7886321015037847"/>
+            <inertia ixx="0.000269" iyy="0.000272" izz="0.000333" ixy="0.0" iyz="0.0" ixz="-1e-06"/>
+        </inertial>
+        <visual>
+            <origin xyz="-0.11007 -3.2e-05 -0.028463" rpy="0 0 0"/>
+            <geometry>
+                <mesh filename="file://$(find two_wheels_core_description)/meshes/lidar_link.stl"
+                      scale="0.001 0.001 0.001"/>
+            </geometry>
+            <material name="silver"/>
+        </visual>
+        <collision>
+            <origin xyz="-0.11007 -3.2e-05 -0.028463" rpy="0 0 0"/>
+            <geometry>
+                <mesh filename="file://$(find two_wheels_core_description)/meshes/lidar_link.stl"
+                      scale="0.001 0.001 0.001"/>
+            </geometry>
+        </collision>
+    </link>
+    <joint name="lidar_link_joint" type="fixed">
+        <origin xyz="0.11007 3.2e-05 0.028463" rpy="0 0 0"/>
+        <parent link="base_link"/>
+        <child link="lidar_link"/>
+    </joint>
     <link name="base_footprint"/>
     <joint name="base_footprint_joint" type="fixed">

Commit message: colors

File: two_wheels_core/urdf/gazebo/gazebo.xacro (robot description, xacro)
@@ -1,7 +1,8 @@
 <?xml version="1.0" encoding="UTF-8"?>
 <robot xmlns:xacro="http://www.ros.org/wiki/xacro">
-    <xacro:property name="body_color" value="Gazebo/Silver"/>
+    <xacro:property name="black" value="Gazebo/Silver"/>
+    <xacro:property name="black" value="Gazebo/Black"/>
     <gazebo reference="base_link">
-        <material>${body_color}</material>
+        <material>${silver}</material>
         <mu1>0.2</mu1>
         <mu2>0.2</mu2>
@@ -10,5 +11,5 @@
     </gazebo>
     <gazebo reference="front_left_wheel">
-        <material>${body_color}</material>
+        <material>${black}</material>
         <mu1>0.2</mu1>
         <mu2>0.2</mu2>
@@ -16,5 +17,5 @@
     </gazebo>
     <gazebo reference="rear_left_wheel">
-        <material>${body_color}</material>
+        <material>${black}</material>
         <mu1>0.2</mu1>
         <mu2>0.2</mu2>
@@ -22,5 +23,5 @@
     </gazebo>
     <gazebo reference="rear_right_wheel">
-        <material>${body_color}</material>
+        <material>${black}</material>
         <mu1>0.2</mu1>
         <mu2>0.2</mu2>
@@ -28,5 +29,5 @@
     </gazebo>
     <gazebo reference="front_right_wheel">
-        <material>${body_color}</material>
+        <material>${black}</material>
         <mu1>0.2</mu1>
         <mu2>0.2</mu2>
@@ -34,5 +35,5 @@
     </gazebo>
     <gazebo reference="lidar_link">
-        <material>${body_color}</material>
+        <material>${black}</material>
         <mu1>0.2</mu1>
         <mu2>0.2</mu2>

File: two_wheels_core/urdf/materials.xacro (robot description, xacro)
@@ -4,3 +4,6 @@
         <color rgba="0.700 0.700 0.700 1.000"/>
     </material>
+    <material name="black">
+        <color rgba="0.0 0.0 0.0 1.000"/>
+    </material>
 </robot>

File: two_wheels_core/urdf/robot_core.xacro (robot description, xacro)
@@ -34,5 +34,5 @@
                       scale="0.001 0.001 0.001"/>
             </geometry>
-            <material name="silver"/>
+            <material name="black"/>
         </visual>
         <collision>
@@ -56,5 +56,5 @@
                       scale="0.001 0.001 0.001"/>
             </geometry>
-            <material name="silver"/>
+            <material name="black"/>
         </visual>
         <collision>
@@ -78,5 +78,5 @@
                       scale="0.001 0.001 0.001"/>
             </geometry>
-            <material name="silver"/>
+            <material name="black"/>
         </visual>
         <collision>
@@ -100,5 +100,5 @@
                       scale="0.001 0.001 0.001"/>
             </geometry>
-            <material name="silver"/>
+            <material name="black"/>
         </visual>
         <collision>
@@ -146,5 +146,5 @@
                       scale="0.001 0.001 0.001"/>
             </geometry>
-            <material name="silver"/>
+            <material name="black"/>
         </visual>
         <collision>

Commit message: fixed gazebo color

File: two_wheels_core/urdf/gazebo/gazebo.xacro (robot description, xacro)
@@ -1,5 +1,5 @@
 <?xml version="1.0" encoding="UTF-8"?>
 <robot xmlns:xacro="http://www.ros.org/wiki/xacro">
-    <xacro:property name="black" value="Gazebo/Silver"/>
+    <xacro:property name="silver" value="Gazebo/Silver"/>
     <xacro:property name="black" value="Gazebo/Black"/>
     <gazebo reference="base_link">
